Commit message: Fixed arm orientation

File: src/full_robot/urdf/ur3e_with_rg2.urdf.xacro (robot description, xacro)
@@ -12,5 +12,5 @@
   <!-- joints required to connect  -->
   <joint name="er5_to_ur3e" type="fixed">
-    <origin xyz="0 0 0" rpy="0 0 0"/>
+    <origin xyz="0 0 0" rpy="0 0 -1.57"/>
     <parent link="er5_body_link"/>
     <child link="base_link"/>
