Commit message: Simplified collision objects, fixed connection to robot

File: src/full_robot/urdf/rg2.urdf.xacro (robot description, xacro)
@@ -21,7 +21,7 @@
       </visual>
       <collision>
-        <origin rpy="0 1.57 0" xyz="0.051 0.0085 0.0015"/>
+        <origin rpy="0 1.57 0" xyz="0.1 0.0085 0.0"/>
         <geometry>
-          <mesh filename="package://full_robot/meshes/rg2_gripper/rg2_.stl" scale="0.001 0.001 0.001"/>
+          <cylinder length="0.2" radius="0.05"/>
         </geometry>
       </collision>

File: src/full_robot/urdf/ur3e_with_rg2.urdf.xacro (robot description, xacro)
@@ -17,5 +17,5 @@
   </joint>
   <joint name="ur3e_to_gripper" type="fixed">
-    <origin xyz="0 0 0" rpy="0 0 0"/>
+    <origin xyz="0 0 0.0" rpy="0 0 0"/>
     <parent link="tool0"/>
     <child link="gripper_extender_link"/>
